Commit message: nav2

File: urdf/robot_2.urdf.xacro (robot description, xacro)
@@ -1,24 +1,40 @@
 <?xml version="1.0"?>
 <robot xmlns:xacro="http://www.ros.org/wiki/xacro" name="hubba">
-<!--
-    <gazebo>
-        <plugin name="differential_drive_linkage" filename="libgazebo_ros_differential_gear.so">
-            <joint_1>base_to_sag_legmil</joint_1>
-            <joint_2>base_to_sol_legmil</joint_2>
-            <differential_joint>base_to_diff_bar</differential_joint>
-            <gear_ratio>1.0</gear_ratio>
-        </plugin>
-    </gazebo> -->
+    <material name="white">
+        <color rgba="1 1 1 1"/>
+    </material>
     <material name="yellow">
         <color rgba="1 1 0 1"/>
     </material>
-    <material name="red">
-        <color rgba="0 0 1 1"/>
-    </material>
+    <material name="vine_red">
+        <color rgba="0.5 0.0 0.1 1.0"/>
+    </material>
+    <material name="indigo">
+        <color rgba="0.29 0.0 0.51 1.0"/>
+    </material>
+    <material name="metallic_grey">
+        <color rgba="0.5 0.5 0.5 1.0"/>
+    </material>
+    <material name="transparent_black">
+        <color rgba="1.0 0.5 0.0 1.0"/>
+    </material>
+    <material name="mint_green">
+        <color rgba="0.6 1.0 0.8 1.0"/>
+    </material>
+    <material name="black">
+        <color rgba="0 0 0 1"/>
+    </material>
+<link name="base_footprint"/>
+    <joint name="base_footprint_to_base_link" type="fixed">
+        <parent link="base_footprint"/>
+        <child link="base_link"/>
+        <origin xyz="0 0 0.0" rpy="0 0 ${-pi/2}"/>
+    </joint>
+<!-- ${pi/2} -->
     <link name="base_link">
         <visual>
             <geometry><box size="0.64 0.98 0.3" /></geometry>
             <origin xyz="0 0 0.60" rpy="0 0 0" />
-            <material name="yellow" />
+            <material name="transparent_black" />
         </visual>
         <collision>
@@ -33,31 +49,27 @@
     </link>
     <gazebo reference="base_link">
-        <material>Gazebo/Yellow</material>
-    </gazebo>
+        <material>Gazebo/Orange</material> </gazebo>
     <link name="diff_bar">
         <visual>
-            <geometry><box size="0.85 0.05 0.05" /></geometry>
+            <geometry><box size="0.05 0.85 0.05" /></geometry>
             <origin xyz="0 0 0" rpy="0 0 0" />
-            <material name="red" />
+            <material name="metallic_grey" />
         </visual>
         <collision>
-            <geometry><box size="0.85 0.05 0.05" /></geometry>
+            <geometry><box size="0.05 0.85 0.05" /></geometry>
             <origin xyz="0 0 0" rpy="0 0 0" />
         </collision>
         <inertial>
-            <mass value="2.0"/>
-            <inertia ixx="0.1" ixy="0" ixz="0" iyy="0.01" iyz="0" izz="0.1"/>
+            <mass value="0.5"/>
+            <inertia ixx="0.03" ixy="0" ixz="0" iyy="0.001" iyz="0" izz="0.03"/>
         </inertial>
     </link>
-    <gazebo reference="diff_bar">
-        <material>Gazebo/Blue</material>
-    </gazebo>
-    <joint name="base_to_diff_bar" type="revolute">
+    <gazebo reference="diff_bar"><material>Gazebo/Grey</material></gazebo>
+    <joint name="base_to_diff_bar" type="fixed">
         <parent link="base_link"/>
         <child link="diff_bar"/>
         <origin xyz="0 0 0.40" rpy="0 0 0"/>
-        <axis xyz="0 0 1"/>
-        <limit lower="-0.5" upper="0.5" effort="1000" velocity="1.0"/>
-        <dynamics damping="1.0" friction="1.0"/>
+        <!-- <axis xyz="0 1 0"/>
+        <limit lower="-0.4" upper="0.4" effort="100" velocity="1.0"/>  -->
     </joint>
     <xacro:macro name="wheel_assembly" params="prefix suffix parent_link reflect_x reflect_y">
@@ -65,5 +77,5 @@
             <visual>
                 <geometry><box size="0.125 0.15 0.11" /></geometry>
-                <material name="yellow" />
+                <material name="mint_green" />
             </visual>
             <collision>
@@ -75,9 +87,8 @@
             </inertial>
         </link>
-        <gazebo reference="${prefix}_${suffix}_kutu"><material>Gazebo/Yellow</material></gazebo>
         <link name="${prefix}_${suffix}_gearbox">
             <visual>
                 <geometry><box size="0.08 0.10 0.055" /></geometry>
-                <material name="yellow" />
+                <material name="indigo" />
             </visual>
             <collision>
@@ -89,10 +100,9 @@
             </inertial>
         </link>
-        <gazebo reference="${prefix}_${suffix}_gearbox"><material>Gazebo/Yellow</material></gazebo>
         <link name="${prefix}_${suffix}_mil">
             <visual>
                 <geometry><cylinder radius="0.01" length="0.12"/></geometry>
                 <origin xyz="0 0 0" rpy="0 0 ${pi/2}" />
-                <material name="red" />
+                <material name="yellow" />
             </visual>
             <collision>
@@ -105,9 +115,8 @@
             </inertial>
         </link>
-        <gazebo reference="${prefix}_${suffix}_mil"><material>Gazebo/Blue</material></gazebo>
         <link name="${prefix}_${suffix}_steering">
             <visual>
                 <geometry><box size="0.16 0.05 0.03" /></geometry>
-                <material name="yellow" />
+                <material name="mint_green" />
             </visual>
             <collision>
@@ -119,9 +128,8 @@
             </inertial>
         </link>
-        <gazebo reference="${prefix}_${suffix}_steering"><material>Gazebo/Yellow</material></gazebo>
         <link name="${prefix}_${suffix}_drive_prf">
             <visual>
                 <geometry><box size="0.07 0.05 0.15" /></geometry>
-                <material name="yellow" />
+                <material name="mint_green" />
             </visual>
             <collision>
@@ -133,10 +141,9 @@
             </inertial>
         </link>
-        <gazebo reference="${prefix}_${suffix}_drive_prf"><material>Gazebo/Yellow</material></gazebo>
         <link name="${prefix}_${suffix}_wheel">
             <visual>
                 <geometry><cylinder radius="0.09" length="0.12"/></geometry>
                 <origin xyz="0 0 0" rpy="0 ${pi/2} 0" />
-                <material name="yellow" />
+                <material name="vine_red" />
             </visual>
             <collision>
@@ -151,9 +158,9 @@
         </link>
         <gazebo reference="${prefix}_${suffix}_wheel">
-            <material>Gazebo/Black</material>
+            <material>Gazebo/Red</material>
             <mu1>1.0</mu1>
             <mu2>1.0</mu2>
             <kp>1000000.0</kp>
-            <kd>1.0</kd>
+            <kd>10000.0</kd>
         </gazebo>
         <joint name="${parent_link}_to_${prefix}_${suffix}_kutu" type="fixed">
@@ -195,5 +202,5 @@
                 <geometry><cylinder radius="0.03" length="0.1"/></geometry>
                 <origin xyz="0 0 0" rpy="0 ${pi/2} 0" />
-                <material name="yellow" />
+                <material name="white" />
             </visual>
             <collision>
@@ -206,9 +213,8 @@
             </inertial>
         </link>
-        <gazebo reference="${prefix}_legmil"><material>Gazebo/Yellow</material></gazebo>
         <link name="${prefix}_prfleg">
             <visual>
                 <geometry><box size="0.12 0.12 0.17" /></geometry>
-                <material name="yellow" />
+                <material name="mint_green" />
             </visual>
             <collision>
@@ -220,10 +226,9 @@
             </inertial>
         </link>
-        <gazebo reference="${prefix}_prfleg"><material>Gazebo/Yellow</material></gazebo>
         <link name="${prefix}_bacak">
             <visual>
                 <geometry><cylinder radius="0.04" length="0.85"/></geometry>
                 <origin xyz="0 0 0" rpy="${pi/2} 0 0" />
-                <material name="yellow" />
+                <material name="metallic_grey" />
             </visual>
             <collision>
@@ -236,11 +241,9 @@
             </inertial>
         </link>
-        <gazebo reference="${prefix}_bacak"><material>Gazebo/Yellow</material></gazebo>
-        <joint name="base_to_${prefix}_legmil" type="continuous">
+        <joint name="base_to_${prefix}_legmil" type="fixed">
             <parent link="base_link"/>
             <child link="${prefix}_legmil"/>
             <origin xyz="${0.39 * reflect_y} 0 0.57" rpy="0 0 0"/>
-            <axis xyz="1 0 0"/>
-            <dynamics damping="0.5" friction="0.5"/>
+            <!-- <axis xyz="1 0 0"/>  -->
         </joint>
         <joint name="${prefix}_legmil_to_prf" type="fixed">
@@ -261,4 +264,130 @@
     <xacro:wheel_assembly prefix="sol" suffix="on" parent_link="sol_bacak" reflect_x="1" reflect_y="-1" />
     <xacro:wheel_assembly prefix="sol" suffix="arka" parent_link="sol_bacak" reflect_x="-1" reflect_y="-1" />
+    <link name="zed2_camera_center">
+        <visual>
+            <geometry><box size="0.033 0.175 0.03" /></geometry>
+            <material name="black"/>
+        </visual>
+        <collision>
+            <geometry><box size="0.033 0.175 0.03" /></geometry>
+        </collision>
+        <inertial>
+            <mass value="0.16"/>
+            <inertia ixx="0.0001" ixy="0" ixz="0" iyy="0.0001" iyz="0" izz="0.0001"/>
+        </inertial>
+    </link>
+    <gazebo reference="zed2_camera_center"><material>Gazebo/Black</material></gazebo>
+    <joint name="base_to_zed2" type="fixed">
+        <parent link="base_link"/>
+        <child link="zed2_camera_center"/>
+        <origin xyz="0 0.49 0.6" rpy="0 0 ${pi/2}"/>
+    </joint>
+    <link name="zed2_camera_optical_frame"/>
+    <joint name="zed2_optical_joint" type="fixed">
+        <parent link="zed2_camera_center"/>
+        <child link="zed2_camera_optical_frame"/>
+        <origin xyz="0 0 0" rpy="${-pi/2} 0 ${-pi/2}"/>
+    </joint>
+    <gazebo reference="zed2_camera_center">
+        <sensor type="depth" name="zed2_sensor">
+            <always_on>true</always_on>
+            <update_rate>10.0</update_rate>
+            <camera name="zed2">
+                <horizontal_fov>1.91986</horizontal_fov>
+                <image><width>640</width><height>360</height><format>R8G8B8</format></image>
+                <clip><near>0.3</near><far>20.0</far></clip>
+                <noise><type>gaussian</type><mean>0.0</mean><stddev>0.007</stddev></noise>
+            </camera>
+            <plugin name="zed2_camera_controller" filename="libgazebo_ros_camera.so">
+                <ros>
+                    <namespace>/zed2</namespace>
+                    <remapping>image_raw:=image_raw</remapping>
+                    <remapping>depth/image_raw:=depth/image_raw</remapping>
+                    <remapping>camera_info:=camera_info</remapping>
+                    <remapping>depth/camera_info:=depth/camera_info</remapping>
+                    <remapping>points:=zed2_sensor/points</remapping>
+                </ros>
+                <frame_name>zed2_camera_optical_frame</frame_name>
+                <hack_baseline>0.12</hack_baseline>
+                <min_depth>0.3</min_depth>
+                <max_depth>20.0</max_depth>
+            </plugin>
+        </sensor>
+    </gazebo>
+<gazebo>
+        <plugin name="gazebo_ros_p3d" filename="libgazebo_ros_p3d.so">
+            <ros><remapping>odom:=odom</remapping></ros>
+            <body_name>base_footprint</body_name>
+            <frame_name>odom</frame_name>
+            <update_rate>30.0</update_rate>
+            <xyz_offset>0 0 0</xyz_offset>
+            <rpy_offset>0 0 0</rpy_offset>
+            <gaussian_noise>0.0</gaussian_noise>
+            <publish_tf>true</publish_tf>
+        </plugin>
+    </gazebo>
+    <!-- <link name="laser_frame">
+        <visual>
+            <geometry>
+                <cylinder radius="0.05" length="0.04"/>
+            </geometry>
+            <material name="black"/>
+        </visual>
+        <collision>
+            <geometry>
+                <cylinder radius="0.05" length="0.04"/>
+            </geometry>
+        </collision>
+        <inertial>
+            <mass value="0.2"/>
+            <inertia ixx="0.001" ixy="0" ixz="0" iyy="0.001" iyz="0" izz="0.001"/>
+        </inertial>
+    </link>
+    <joint name="laser_joint" type="fixed">
+        <parent link="base_link"/>
+        <child link="laser_frame"/>
+        <origin xyz="0 0 0.8" rpy="0 0 ${pi/2}"/> </joint>
+    <gazebo reference="laser_frame">
+        <material>Gazebo/Black</material>
+        <sensor name="lidar" type="ray">
+            <always_on>true</always_on>
+            <visualize>true</visualize> <update_rate>10.0</update_rate>
+            <ray>
+                <scan>
+                    <horizontal>
+                        <samples>360</samples>
+                        <resolution>1.0</resolution>
+                        <min_angle>-3.14159</min_angle>
+                        <max_angle>3.14159</max_angle>
+                    </horizontal>
+                </scan>
+                <range>
+                    <min>0.15</min>
+                    <max>12.0</max>
+                    <resolution>0.015</resolution>
+                </range>
+                <noise>
+                    <type>gaussian</type>
+                    <mean>0.0</mean>
+                    <stddev>0.01</stddev>
+                </noise>
+            </ray>
+            <plugin name="scan" filename="libgazebo_ros_ray_sensor.so">
+                <ros>
+                    <remapping>~/out:=scan</remapping>
+                </ros>
+                <output_type>sensor_msgs/LaserScan</output_type>
+                <frame_name>laser_frame</frame_name>
+            </plugin>
+        </sensor>
+    </gazebo> -->
+    <!-- <gazebo>
+        <plugin name="differential_weight_averager" filename="libgazebo_ros_differential_gear.so">
+            <joint_1>base_to_sag_legmil</joint_1>
+            <joint_2>base_to_sol_legmil</joint_2>
+            <differential_joint>base_to_diff_bar</differential_joint>
+            <gear_ratio>1.0</gear_ratio>
+        </plugin>
+    </gazebo> -->
     <ros2_control name="GazeboSystem" type="system">
         <hardware>
@@ -268,16 +397,20 @@
             <command_interface name="velocity"/>
             <state_interface name="velocity"/>
+            <state_interface name="position"/>
          </joint>
         <joint name="sag_on_drive_to_wheel">
             <command_interface name="velocity"/>
             <state_interface name="velocity"/>
+            <state_interface name="position"/>
         </joint>
         <joint name="sol_arka_drive_to_wheel">
             <command_interface name="velocity"/>
             <state_interface name="velocity"/>
+            <state_interface name="position"/>
         </joint>
         <joint name="sag_arka_drive_to_wheel">
             <command_interface name="velocity"/>
             <state_interface name="velocity"/>
+            <state_interface name="position"/>
         </joint>
         <joint name="sol_on_gearbox_to_mil">

Commit message: Update robot_2.urdf.xacro

File: urdf/robot_2.urdf.xacro (robot description, xacro)
@@ -69,5 +69,5 @@
         <parent link="base_link"/>
         <child link="diff_bar"/>
-        <origin xyz="0 0 0.40" rpy="0 0 0"/>
+        <origin xyz="0 0 0.40" rpy="0 0 ${pi/2}"/>
         <!-- <axis xyz="0 1 0"/>
         <limit lower="-0.4" upper="0.4" effort="100" velocity="1.0"/>  -->
