Commit message: a

File: urdf/robot_2_real.urdf.xacro (robot description, xacro)
@@ -34,10 +34,10 @@
     <link name="base_link">
         <visual>
-            <geometry><box size="0.64 0.98 0.3" /></geometry>
+            <geometry><box size="0.46 0.85 0.3" /></geometry>
             <origin xyz="0 0 0.60" rpy="0 0 0" />
             <material name="transparent_black" />
         </visual>
         <collision>
-            <geometry><box size="0.64 0.98 0.3" /></geometry>
+            <geometry><box size="0.46 0.85 0.3" /></geometry>
             <origin xyz="0 0 0.60" rpy="0 0 0" />
         </collision>
@@ -52,10 +52,10 @@
     <link name="diff_bar">
         <visual>
-            <geometry><box size="0.05 0.85 0.05" /></geometry>
+            <geometry><box size="0.05 0.50 0.05" /></geometry>
             <origin xyz="0 0 0" rpy="0 0 0" />
             <material name="metallic_grey" />
         </visual>
         <collision>
-            <geometry><box size="0.05 0.85 0.05" /></geometry>
+            <geometry><box size="0.05 0.50 0.05" /></geometry>
             <origin xyz="0 0 0" rpy="0 0 0" />
         </collision>
@@ -167,5 +167,5 @@
             <parent link="${parent_link}"/>
             <child link="${prefix}_${suffix}_kutu"/>
-            <origin xyz="0 ${0.485 * reflect_x} -0.025" rpy="0 0 0"/>
+            <origin xyz="0 ${0.4925 * reflect_x} -0.025" rpy="0 0 0"/>
         </joint>
         <joint name="${prefix}_${suffix}_kutu_to_gearbox" type="fixed">
@@ -228,10 +228,10 @@
         <link name="${prefix}_bacak">
             <visual>
-                <geometry><cylinder radius="0.04" length="0.85"/></geometry>
+                <geometry><cylinder radius="0.04" length="0.835"/></geometry>
                 <origin xyz="0 0 0" rpy="${pi/2} 0 0" />
                 <material name="metallic_grey" />
             </visual>
             <collision>
-                <geometry><cylinder radius="0.04" length="0.85"/></geometry>
+                <geometry><cylinder radius="0.04" length="0.835"/></geometry>
                 <origin xyz="0 0 0" rpy="${pi/2} 0 0" />
             </collision>
@@ -244,5 +244,5 @@
             <parent link="base_link"/>
             <child link="${prefix}_legmil"/>
-            <origin xyz="${0.36 * reflect_y} 0 0.57" rpy="0 0 0"/>
+            <origin xyz="${0.25 * reflect_y} 0 0.57" rpy="0 0 0"/>
             <!-- <axis xyz="1 0 0"/>  -->
         </joint>
